Commit message: Completed base of adrover

File: description/robot.urdf.xacro (robot description, xacro)
@@ -1,5 +1,4 @@
 <?xml version="1.0"?>
 <robot xmlns:xacro="http://www.ros.org/wiki/xacro"  name="Adrover">
-    <!-- Example link -->
-    <link name="base_link"></link>
+    <xacro:include filename="robot_core.xacro"/>
 </robot>

Commit message: Adrover_gazebo_control_world upate

File: description/robot.urdf.xacro (robot description, xacro)
@@ -2,3 +2,4 @@
 <robot xmlns:xacro="http://www.ros.org/wiki/xacro"  name="Adrover">
     <xacro:include filename="robot_core.xacro"/>
+    <xacro:include filename="gazebo_control.xacro"/>
 </robot>

File: description/robot_core.xacro (robot description, xacro)
@@ -43,4 +43,7 @@
             <origin xyz="0.295 0.0 0.15"/>
         </xacro:inertial_box>
+        <!-- <gazebo reference="chassis">
+            <material>Gazebo/Black</material>
+        </gazebo> -->
         <visual>
             <origin xyz="0.295 0.245 0.15"/>
@@ -59,4 +62,7 @@
             <origin xyz="0.295 0.245 0.15"/>
         </xacro:inertial_box>
+        <!-- <gazebo reference="chassis">
+            <material>Gazebo/Black</material>
+        </gazebo> -->
         <visual>
             <origin xyz="0.295 -0.245 0.15"/>
@@ -75,4 +81,7 @@
             <origin xyz="0.295 -0.245 0.15"/>
         </xacro:inertial_box>
+        <!-- <gazebo reference="chassis">
+            <material>Gazebo/Black</material>
+        </gazebo> -->
         <visual>
             <origin xyz="0.0 0.0 0.15"/>
@@ -91,4 +100,7 @@
             <origin xyz="0.0 0.0 0.15"/>
         </xacro:inertial_box>
+        <!-- <gazebo reference="chassis">
+            <material>Gazebo/Black</material>
+        </gazebo> -->
         <visual>
             <origin xyz="0.59 0.0 0.15"/>
@@ -107,4 +119,7 @@
             <origin xyz="0.59 0.0 0.15"/>
         </xacro:inertial_box>
+        <gazebo reference="chassis">
+            <material>Gazebo/Black</material>
+        </gazebo>
     </link>
     <!-- Left wheel -->
@@ -130,4 +145,7 @@
             <origin xyz="0.0 0.0 0.0" rpy="0.0 0.0 0.0"/>
         </xacro:inertial_cylinder>
+        <gazebo reference="left_wheel_link">
+            <material>Gazebo/Orange</material>
+        </gazebo>
     </link>
     <!-- Right wheel -->
@@ -153,4 +171,7 @@
             <origin xyz="0.0 0.0 0.0" rpy="0.0 0.0 0.0"/>
         </xacro:inertial_cylinder>
+        <gazebo reference="right_wheel_link">
+            <material>Gazebo/Orange</material>
+        </gazebo>
     </link>
     <!-- Caster wheel 1 -->
@@ -177,4 +198,9 @@
             <origin xyz="0.0 0.0 0.0" rpy="0.0 0.0 0.0"/>
         </xacro:inertial_sphere>
+        <gazebo reference="caster_wheel_link_1">
+            <material>Gazebo/White</material>
+            <mu1 value="0.001"/>
+            <mu2 value="0.001"/>
+        </gazebo>
     </link>
     <!-- Caster wheel 2 -->
@@ -201,4 +227,9 @@
             <origin xyz="0.0 0.0 0.0" rpy="0.0 0.0 0.0"/>
         </xacro:inertial_sphere>
+        <gazebo reference="caster_wheel_link_2">
+            <material>Gazebo/White</material>
+            <mu1 value="0.001"/>
+            <mu2 value="0.001"/>
+        </gazebo>
     </link>
     <!-- Caster wheel 3 -->
@@ -225,4 +256,9 @@
             <origin xyz="0.0 0.0 0.0" rpy="0.0 0.0 0.0"/>
         </xacro:inertial_sphere>
+        <gazebo reference="caster_wheel_link_3">
+            <material>Gazebo/White</material>
+            <mu1 value="0.001"/>
+            <mu2 value="0.001"/>
+        </gazebo>
     </link>
     <!-- Caster wheel 4 -->
@@ -249,4 +285,9 @@
             <origin xyz="0.0 0.0 0.0" rpy="0.0 0.0 0.0"/>
         </xacro:inertial_sphere>
+        <gazebo reference="caster_wheel_link_4">
+            <material>Gazebo/White</material>
+            <mu1 value="0.001"/>
+            <mu2 value="0.001"/>
+        </gazebo>
     </link>
 </robot>

Commit message: Made the adrover to view in rviz

File: description/robot.urdf.xacro (robot description, xacro)
@@ -1,5 +1,4 @@
 <?xml version="1.0"?>
 <robot xmlns:xacro="http://www.ros.org/wiki/xacro"  name="Adrover">
-    <!-- Example link -->
-    <link name="base_link"></link>
+    <xacro:include filename="robot_core.xacro" />
 </robot>

Commit message: LiDAR integration

File: description/robot.urdf.xacro (robot description, xacro)
@@ -2,3 +2,5 @@
 <robot xmlns:xacro="http://www.ros.org/wiki/xacro"  name="Adrover">
     <xacro:include filename="robot_core.xacro" />
+    <xacro:include filename="gazebo_control.xacro" />
+    <xacro:include filename="lidar.xacro" />
 </robot>

File: description/robot_core.xacro (robot description, xacro)
@@ -44,5 +44,5 @@
     </link>
     <gazebo reference="chassis_link_left">
-        <material>Gazebo/White</material>
+        <material>Gazebo/Black</material>
     </gazebo>
     <!-- Chassis right -->
@@ -70,4 +70,7 @@
         </xacro:inertial_box>
     </link>
+    <gazebo reference="chassis_link_right">
+        <material>Gazebo/Black</material>
+    </gazebo>
     <!-- Chassis front -->
     <joint name="chassis_joint_front" type="fixed">
@@ -94,4 +97,7 @@
         </xacro:inertial_box>
     </link>
+    <gazebo reference="chassis_link_front">
+        <material>Gazebo/Black</material>
+    </gazebo>
     <!-- Chassis back -->
     <joint name="chassis_joint_back" type="fixed">
@@ -118,4 +124,7 @@
         </xacro:inertial_box>
     </link>
+    <gazebo reference="chassis_link_back">
+        <material>Gazebo/Black</material>
+    </gazebo>
     <!-- Left Wheel -->
     <joint name="left_wheel_joint" type="continuous">
@@ -143,4 +152,7 @@
         </xacro:inertial_cylinder>
     </link>
+    <gazebo reference="left_wheel_link">
+        <material>Gazebo/Red</material>
+    </gazebo>
     <!-- Right wheel -->
     <joint name="right_wheel_joint" type="continuous">
@@ -168,4 +180,7 @@
         </xacro:inertial_cylinder>
     </link>
+    <gazebo reference="right_wheel_link">
+        <material>Gazebo/Red</material>
+    </gazebo>
     <!-- Caster wheel left front -->
     <joint name="caster_wheel_joint_lf" type="fixed">
@@ -192,4 +207,9 @@
         </xacro:inertial_sphere>
     </link>
+    <gazebo reference="caster_wheel_link_lf">
+        <material>Gazebo/Green</material>
+        <mu1 value="0.001"/>
+        <mu2 value="0.001"/>
+    </gazebo>
     <!-- Caster wheel right front -->
     <joint name="caster_wheel_joint_rf" type="fixed">
@@ -216,4 +236,9 @@
         </xacro:inertial_sphere>
     </link>
+    <gazebo reference="caster_wheel_link_rf">
+        <material>Gazebo/Green</material>
+        <mu1 value="0.001"/>
+        <mu2 value="0.001"/>
+    </gazebo>
     <!-- Caster wheel left back -->
     <joint name="caster_wheel_joint_lb" type="fixed">
@@ -240,4 +265,9 @@
         </xacro:inertial_sphere>
     </link>
+    <gazebo reference="caster_wheel_link_lb">
+        <material>Gazebo/Green</material>
+        <mu1 value="0.001"/>
+        <mu2 value="0.001"/>
+    </gazebo>
     <!-- Caster wheel right back -->
     <joint name="caster_wheel_joint_rb" type="fixed">
@@ -264,4 +294,9 @@
         </xacro:inertial_sphere>
     </link>
+    <gazebo reference="caster_wheel_link_rb">
+        <material>Gazebo/Green</material>
+        <mu1 value="0.001"/>
+        <mu2 value="0.001"/>
+    </gazebo>
     <!-- LCD -->
     <joint name="lcd_joint" type="fixed">
@@ -288,3 +323,6 @@
         </xacro:inertial_box>
     </link>
+    <gazebo reference="lcd_link">
+        <material>Gazebo/Blue</material>
+    </gazebo>
 </robot>
