Commit message: ros_control, camera and lidar integrated

File: description/lidar.xacro (robot description, xacro)
@@ -25,7 +25,8 @@
     </link>
     <gazebo reference="laser_frame">
+        <material>Gazebo/White</material>
         <sensor name="laser" type="ray">
             <pose> 0 0 0 0 0 0 </pose>
-            <visualize>true</visualize>
+            <visualize>false</visualize>
             <update_rate>10</update_rate>
             <ray>

File: description/robot.urdf.xacro (robot description, xacro)
@@ -4,3 +4,4 @@
     <xacro:include filename="gazebo_control.xacro" />
     <xacro:include filename="lidar.xacro" />
+    <xacro:include filename="camera.xacro" />
 </robot>

Commit message: adrover working simulation

File: description/lidar.xacro (robot description, xacro)
@@ -14,13 +14,4 @@
             <material name="white"/>
         </visual>
-        <collision>
-            <origin xyz="0.0 0.0 0.0" rpy="0.0 0.0 0.0"/>
-            <geometry>
-                <cylinder radius="0.06" length="0.035"/>
-            </geometry>
-        </collision>
-        <xacro:inertial_cylinder mass="0.1" radius="0.06" length="0.035">
-            <origin xyz="0.0 0.0 0.0" rpy="0.0 0.0 0.0"/>
-        </xacro:inertial_cylinder>
     </link>
     <gazebo reference="laser_frame">
@@ -28,6 +19,6 @@
         <sensor name="laser" type="ray">
             <pose> 0 0 0 0 0 0 </pose>
-            <visualize>false</visualize>
-            <update_rate>10</update_rate>
+            <visualize>true</visualize>
+            <update_rate>100</update_rate>
             <ray>
                 <scan>
@@ -40,7 +31,7 @@
                 </scan>
                 <range>
-                    <min>0.3</min>
+                    <min>0.15</min>
                     <max>12</max>
-                    <resolution>0.01</resolution>
+                    <resolution>0.001</resolution>
                 </range>
             </ray>
