Commit message: PI configuration

File: description/ros2_control.xacro (robot description, xacro)
@@ -1,5 +1,33 @@
 <?xml version="1.0"?>
 <robot xmlns:xacro="http://www.ros.org/wiki/xacro">
-    <ros2_control name="GazeboSystem" type="system">
+    <ros2_control name="RealRobot" type="SystemInterface">
+        <hardware>
+            <plugin>diffdrive_arduino/DiffDriveArduino</plugin>
+            <param name="left_wheel_names">left_wheel_joint</param>
+            <param name="right_wheel_names">right_wheel_joint</param>
+            <param name="loop_rate">100</param>
+            <param name="device">/dev/serial/by-id/usb-1a86_USB2.0-Ser_-if00-port0</param>
+            <param name="baud_rate">57600</param>
+            <param name="timeout_ms">1000</param>
+            <param name="enc_counts_per_rev">8400</param>
+        </hardware>
+        <joint name="left_wheel_joint">
+            <command_interface name="velocity">
+                <param name="min">-10</param>
+                <param name="max">10</param>
+            </command_interface>
+            <state_interface name="velocity" />
+            <state_interface name="position" />
+        </joint>
+        <joint name="right_wheel_joint">
+            <command_interface name="velocity">
+                <param name="min">-10</param>
+                <param name="max">10</param>
+            </command_interface>
+            <state_interface name="velocity" />
+            <state_interface name="position" />
+        </joint>
+    </ros2_control>
+    <!-- <ros2_control name="GazeboSystem" type="system">
         <hardware>
             <plugin>gazebo_ros2_control/GazeboSystem</plugin>
@@ -10,6 +38,6 @@
                 <param name="max">10</param>
             </command_interface>
+            <state_interface name="velocity" />
             <state_interface name="position" />
-            <state_interface name="velocity" />
         </joint>
         <joint name="right_wheel_joint">
@@ -18,8 +46,8 @@
                 <param name="max">10</param>
             </command_interface>
+            <state_interface name="velocity" />
             <state_interface name="position" />
-            <state_interface name="velocity" />
         </joint>
-    </ros2_control>
+    </ros2_control> -->
     <gazebo>
         <plugin name="gazebo_ros2_control" filename="libgazebo_ros2_control.so">
