Commit message: Started adding colors to the gazebo rover. Made launch file for robot visualizing

File: description/robot_core.xacro (robot description, xacro)
@@ -43,4 +43,7 @@
         </xacro:inertial_box>
     </link>
+    <gazebo reference="chassis_link_left">
+        <material>Gazebo/White</material>
+    </gazebo>
     <!-- Chassis right -->
     <joint name="chassis_joint_right" type="fixed">

Commit message: loads the model in gazebo. The model falls down

File: description/robot_core.xacro (robot description, xacro)
@@ -324,3 +324,30 @@
         <material>Gazebo/Blue</material>
     </gazebo>
+    <!-- LCD Support -->
+    <joint name="lcd_support_joint" type="fixed">
+        <origin xyz="0.0 0.0 0.36" rpy="0.0 0.0 0.0"/>
+        <parent link="chassis_link_back"/>
+        <child link="lcd_support_link"/>
+    </joint>
+    <link name="lcd_support_link">
+        <visual name="">
+            <origin xyz="0.15 0.0 0.43" rpy="0.0 -2.79 0.0"/>
+            <geometry>
+                <box size="0.06 0.43 0.86"/>
+            </geometry>
+            <material name="blue" />
+        </visual>
+        <collision>
+            <origin xyz="0.15 0.0 0.43" rpy="0.0 -2.79 0.0"/>
+            <geometry>
+                <box size="0.06 0.43 0.86"/>
+            </geometry>
+        </collision>
+        <xacro:inertial_box mass="0.5" x="0.06" y="0.43" z="0.86">
+            <origin xyz="0.15 0.0 0.43" rpy="0.0 -2.79 0.0"/>
+        </xacro:inertial_box>
+    </link>
+    <gazebo reference="lcd_support_link">
+        <material>Gazebo/Blue</material>
+    </gazebo>
 </robot>

Commit message: Working individual settings of gazebo_control and ros2_control.

File: description/robot_core.xacro (robot description, xacro)
@@ -144,5 +144,5 @@
         <collision>
             <geometry>
-                <sphere radius="0.6"/>
+                <cylinder radius="0.06" length="0.0005"/>
             </geometry>
         </collision>
@@ -171,5 +171,5 @@
         <collision>
             <geometry>
-                <sphere radius="0.6"/>
+                <cylinder radius="0.06" length="0.0005"/>
             </geometry>
         </collision>
@@ -324,30 +324,3 @@
         <material>Gazebo/Blue</material>
     </gazebo>
-    <!-- LCD Support -->
-    <joint name="lcd_support_joint" type="fixed">
-        <origin xyz="0.0 0.0 0.36" rpy="0.0 0.0 0.0"/>
-        <parent link="chassis_link_back"/>
-        <child link="lcd_support_link"/>
-    </joint>
-    <link name="lcd_support_link">
-        <visual name="">
-            <origin xyz="0.15 0.0 0.43" rpy="0.0 -2.79 0.0"/>
-            <geometry>
-                <box size="0.06 0.43 0.86"/>
-            </geometry>
-            <material name="blue" />
-        </visual>
-        <collision>
-            <origin xyz="0.15 0.0 0.43" rpy="0.0 -2.79 0.0"/>
-            <geometry>
-                <box size="0.06 0.43 0.86"/>
-            </geometry>
-        </collision>
-        <xacro:inertial_box mass="0.5" x="0.06" y="0.43" z="0.86">
-            <origin xyz="0.15 0.0 0.43" rpy="0.0 -2.79 0.0"/>
-        </xacro:inertial_box>
-    </link>
-    <gazebo reference="lcd_support_link">
-        <material>Gazebo/Blue</material>
-    </gazebo>
 </robot>

Commit message: Working rpi code

File: description/robot_core.xacro (robot description, xacro)
@@ -133,4 +133,5 @@
         <axis xyz="0 0 1"/>
         <origin xyz="0.3125 0.1625 0" rpy="-1.5708 0 0"/>
+        <hardwareInterface>  <velocity>  <param name="min">-10.0</param>  <param name="max">10.0</param>  </velocity> </hardwareInterface>
     </joint>
     <link name="left_wheel_link">
@@ -160,4 +161,5 @@
         <axis xyz="0 0 -1"/>
         <origin xyz="0.3125 -0.1625 0" rpy="1.5708 0 0"/>
+        <hardwareInterface>  <velocity>  <param name="min">-10.0</param>  <param name="max">10.0</param>  </velocity> </hardwareInterface>
     </joint>
     <link name="right_wheel_link">

File: description/ros2_control.xacro (robot description, xacro)
@@ -1,15 +1,16 @@
 <?xml version="1.0"?>
 <robot xmlns:xacro="http://www.ros.org/wiki/xacro">
-    <ros2_control name="RealRobot" type="SystemInterface">
+    <ros2_control name="Adrover" type="system">
         <hardware>
             <plugin>diffdrive_arduino/DiffDriveArduino</plugin>
-            <param name="left_wheel_names">left_wheel_joint</param>
-            <param name="right_wheel_names">right_wheel_joint</param>
-            <param name="loop_rate">100</param>
+            <param name="left_wheel_name">left_wheel_joint</param>
+            <param name="right_wheel_name">right_wheel_joint</param>
+            <param name="loop_rate">50</param>
             <param name="device">/dev/serial/by-id/usb-1a86_USB2.0-Ser_-if00-port0</param>
             <param name="baud_rate">57600</param>
-            <param name="timeout_ms">1000</param>
+            <param name="timeout">1000</param>
             <param name="enc_counts_per_rev">8400</param>
         </hardware>
+    <!-- Note everything below here is the same as the Gazebo one -->
         <joint name="left_wheel_joint">
             <command_interface name="velocity">
@@ -17,6 +18,6 @@
                 <param name="max">10</param>
             </command_interface>
-            <state_interface name="velocity" />
-            <state_interface name="position" />
+            <state_interface name="velocity"/>
+            <state_interface name="position"/>
         </joint>
         <joint name="right_wheel_joint">
@@ -25,29 +26,8 @@
                 <param name="max">10</param>
             </command_interface>
-            <state_interface name="velocity" />
-            <state_interface name="position" />
+            <state_interface name="velocity"/>
+            <state_interface name="position"/>
         </joint>
     </ros2_control>
-    <!-- <ros2_control name="GazeboSystem" type="system">
-        <hardware>
-            <plugin>gazebo_ros2_control/GazeboSystem</plugin>
-        </hardware>
-        <joint name="left_wheel_joint">
-            <command_interface name="velocity">
-                <param name="min">-10</param>
-                <param name="max">10</param>
-            </command_interface>
-            <state_interface name="velocity" />
-            <state_interface name="position" />
-        </joint>
-        <joint name="right_wheel_joint">
-            <command_interface name="velocity">
-                <param name="min">-10</param>
-                <param name="max">10</param>
-            </command_interface>
-            <state_interface name="velocity" />
-            <state_interface name="position" />
-        </joint>
-    </ros2_control> -->
     <gazebo>
         <plugin name="gazebo_ros2_control" filename="libgazebo_ros2_control.so">
